File: LED-Driver.kicad_pcb (KiCad board)
At the start: 2 copper layers, 58.2 x 53.5 mm, 9 parts, among them J1 Conn_01x04, J2 Barrel_Jack_Switch, Q1 NTE289, Q2 NTE289, Q3 NTE289, U1 Pico

Commit message: Connect grounds
Routing:
- net GND: track 15.3 -> 55.1 mm
Changed lines of the file:
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@@
 	)
 	(segment
-		(start 36.39 19.92)
-		(end 50.21 19.92)
+		(start 63.75 37.25)
+		(end 63.75 43.75)
 		(width 0.2)
-		(layer "F.Cu")
+		(layer "B.Cu")
 		(net 2)
 	)
 	(segment
-		(start 50.21 19.92)
+		(start 63.75 30.75)
+		(end 63.75 37.25)
+		(width 0.2)
+		(layer "B.Cu")
+		(net 2)
+	)
+	(segment
+		(start 63.75 43.75)
+		(end 65.57 43.75)
+		(width 0.2)
+		(layer "B.Cu")
+		(net 2)
+	)
+	(segment
+		(start 63.75 30.75)
+		(end 65.57 30.75)
+		(width 0.2)
+		(layer "B.Cu")
+		(net 2)
+	)
+	(segment
+		(start 65.57 43.75)
+		(end 65.59 43.73)
+		(width 0.2)
+		(layer "B.Cu")
+		(net 2)
+	)
+	(segment
+		(start 51.29 21)
+		(end 62 21)
+		(width 0.2)
+		(layer "B.Cu")
+		(net 2)
+	)
+	(segment
+		(start 36.39 19.84)
+		(end 50.13 19.84)
+		(width 0.2)
+		(layer "B.Cu")
+		(net 2)
+	)
+	(segment
+		(start 63.75 37.25)
+		(end 65.57 37.25)
+		(width 0.2)
+		(layer "B.Cu")
+		(net 2)
+	)
+	(segment
+		(start 65.57 37.25)
+		(end 65.59 37.23)
+		(width 0.2)
+		(layer "B.Cu")
+		(net 2)
+	)
+	(segment
+		(start 50.13 19.84)
 		(end 51.29 21)
 		(width 0.2)
-		(layer "F.Cu")
+		(layer "B.Cu")
 		(net 2)
 	)
+	(segment
+		(start 63.75 22.75)
+		(end 63.75 30.75)
+		(width 0.2)
+		(layer "B.Cu")
+		(net 2)
+	)
+	(segment
+		(start 62 21)
+		(end 63.75 22.75)
+		(width 0.2)
+		(layer "B.Cu")
+		(net 2)
+	)
+	(segment
+		(start 65.57 30.75)
+		(end 65.59 30.73)
+		(width 0.2)
+		(layer "B.Cu")
+		(net 2)
+	)
